File: designs/wooden_alarm.sch (EAGLE design)
At the start: 20 parts, among them IC1 ESP-12E/F

Commit message: final changes v1 design
Parts:
- added IO_15_SWITCH, IO_2_SWITCH: (no value), con-lstb:MA03-1
Connections:
- removed net N$8: IC1.IO0, IO_0_SWITCH.3, R5.2
- new net N$2: IO_2_SWITCH.3, R4.2
- new net N$5: IO_15_SWITCH.3, R3.1
- new net SWITCH_PIN: IC1.IO13, IO_0_SWITCH.2, R5.2
- net CCW: now also IO_2_SWITCH.1
- net CW: now also IO_15_SWITCH.1
- net GND: now also IO_0_SWITCH.3, JUMPER_TOUCH.3, R3.2; no longer IO_0_SWITCH.2, JUMPER_TOUCH.1, R3.1
- net N$3: now also IO_15_SWITCH.2; no longer R3.2
- net N$7: now also IO_2_SWITCH.2; no longer R4.2
- net SQW: now also IC1.IO0; no longer IC1.IO16
- net SWITCH: now also IO_0_SWITCH.1
- net TOUCH_IO: now also IC1.IO16, JUMPER_TOUCH.1; no longer IC1.IO13, JUMPER_TOUCH.2
- net VCC: now also JUMPER_TOUCH.2; no longer JUMPER_TOUCH.3
Other:
- moved on the sheet: C2, C3, C4, IO_0_SWITCH, JUMPER_ENCODER, R3, R4, R5, R6, R7, R8
